File: organ_ciruit.kicad_sch (KiCad schematic)
At the start: 0 parts

Commit message: hi
Parts:
- added C1: 33nf, symbol Device:C
- added D1, D2, D3, D4, D5, D6, D7, D8, D9: LED, symbol Device:LED
- added LS1: Speaker, symbol Device:Speaker
- added Q1: 2N3904, Package_TO_SOT_THT:TO-92_Inline, symbol Transistor_BJT:2N3904
- added Q2: 2N3906, Package_TO_SOT_THT:TO-92_Inline, symbol Transistor_BJT:2N3906
- added R1: 1k, symbol Device:R
- added R2: 270k, symbol Device:R
- added R3: 20k, symbol Device:R
- added R4, R5: 39k, symbol Device:R
- added R6, R9: 47k, symbol Device:R
- added R7: 22k, symbol Device:R
- added R8: 68k, symbol Device:R
- added SW1, SW2, SW3, SW4, SW5, SW6, SW7, SW8: SW_Push, symbol Switch:SW_Push
- added SW9: slide, Button_Switch_THT:SW_Slide-03_Wuerth-WS-SLTV_10x2.5x6.4_P2.54mm, symbol Switch:SW_Wuerth_450301014042
Connections:
- new net: R4.2, R5.1, SW3.1
- new net: R5.2, R6.1, SW4.1
- new net: R7.2, R8.1, SW6.1
- new net: R8.2, R9.1, SW7.1
- new net: R2.1, R3.1, SW1.1
- new net: R3.2, R4.1, SW2.1
- new net: C1.1, Q1.1 (E), R1.2
- new net: LS1.1, Q1.3 (C), Q2.3 (C)
- new net: R6.2, R7.1, SW5.1
- new net: Q2.2 (B), R1.1
- new net +9V: Q2.1 (E), R2.2, SW9.1 (B)
- new net GND: C1.2, LS1.2, R9.2, SW8.1
- new net jumper: Q1.2 (B), SW1.2, SW2.2, SW3.2, SW4.2, SW5.2, SW6.2, SW7.2, SW8.2

Commit message: hi
Parts:
- removed D9: LED, symbol Device:LED
- added R10, R11, R12, R13, R14, R15, R16, R17: 1k, symbol Device:R
Connections:
- net +9V: now also SW9.3 (A); no longer Q2.1 (E), R2.2, SW9.1 (B)
- net GND: now also D1.1 (K), D2.1 (K), D3.1 (K), D4.1 (K), D5.1 (K), D6.1 (K), D7.1 (K), D8.1 (K), R17.1
- net jumper: now also R3.1, SW1.1, R10.1; no longer SW1.2, SW2.2, SW3.2, SW4.2, SW5.2, SW6.2, SW7.2, SW8.2
- net at R4.2, R5.1, SW3.1: now also R12.1
- net at R5.2, R6.1, SW4.1: now also R13.1
- net at D7.2 (A): now also R11.2
- net at R7.2, R8.1, SW6.1: now also R15.1
- net at R8.2, R9.1, SW7.1: now also R16.1
- net at R3.2, R4.1, SW2.1: now also R11.1
- net at D3.2 (A): now also R15.2
- net at R6.2, R7.1, SW5.1: now also R14.1
- net at D6.2 (A): now also R12.2
- net at D8.2 (A): now also R10.2
- net at D1.2 (A): now also R17.2
- net at D5.2 (A): now also R13.2
- net at D2.2 (A): now also R16.2
- net at D4.2 (A): now also R14.2
- new net: R2.1, SW1.2, SW2.2, SW3.2, SW4.2, SW5.2, SW6.2, SW7.2, SW8.2
- new net power: Q2.1 (E), R2.2, SW9.1 (B)
Other:
- note added: "Keyswitch"
- note added: "Ladder/Jumper"
- note added: "Leds"
- note added: "Organ Circuit - ZYYY"
- note added: "Oscillator Core"
- note added: "Power & Ground"
- moved on the sheet: C1, D1, D2, D3, D4, D5, D6, D7, D8, LS1, Q1, Q2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
